File: Kicad/Images/Images.kicad_sch (KiCad schematic)
At the start: 6 parts, among them U1 Z_{1}=1, U2 Z_{2}=2, U3 L=1, U4 L=1, U5 C=1

Commit message: Added Changes
Parts:
- added R2, R3, R4, R5, R6, R7: Z_{0}, symbol HF_Sym:R
- added R8, R9: R_{x}, symbol HF_Sym:R
- added U10, U7: L, symbol HF_Sym:L
- added U11, U6, U8, U9: C, symbol HF_Sym:C
- added U12, U13, U19, U20: Z_{0}, symbol HF_Sym:UE
- added U14, U18: Z_{1}, symbol HF_Sym:UE
- added U15, U17: L_{1}, symbol HF_Sym:L
- added U16, U21: L/2, symbol HF_Sym:L
- added U22: Z_{1}, symbol HF_Sym:L
- added U23: n:1, symbol HF_Sym:Trafo
- added U24: Z_{2}, symbol HF_Sym:L
- added U26: 1:n, symbol HF_Sym:Trafo
Connections:
- net at U1.: now also U2.
- net at U2.: now also R1.; no longer U1.
- net at U4.: now also U3., U5.
- new net: U1., U2.
- new net: U14., U18.
- new net: U14., U15.
- new net: U14., U16.
- new net: U14., U19.
- new net: U10., U11., U13.
- new net: U10., U12., U9.
- new net: R2., U6., U7.
- new net: R2., R3., U6., U8.
- new net: U24., U26.
- new net: U22., U24.
- new net: R7., U20. (x2)
- new net: R3., U7., U8.
- new net: U11., U12., U13., U9.
- new net: R5., U13. (x2)
- new net: R1., U2.
- new net: U17., U18.
- new net: U18., U20.
- new net: U18., U21.
- new net: U17., U20.
- new net: R6., U19. (x2)
- new net: R4., U12. (x2)
- new net: U22., U26.
- new net: U15., U19.
- new net: U16., U21.
- new net Earth: R8., R9.
- now unconnected: U3., U5.
Other:
- note added: "1"
- note added: "2"
- note added: "3"
- note added: "4"
- note added: "LL"
- note added: "Z_{0}"

Commit message: Added Beispiele
Parts:
- removed U22: Z_{1}, symbol HF_Sym:L
- removed U24: Z_{2}, symbol HF_Sym:L
- removed U26: 1:n, symbol HF_Sym:Trafo
- added R10: Z_{0}, symbol HF_Sym:R
- added U22: C_{11}, symbol HF_Sym:C
- added U24: Z_{12}, symbol HF_Sym:UE
- added U25: C_{3}=1, symbol HF_Sym:C
- added U26: C_{3}, symbol HF_Sym:C
- added U27: L_{1}=1, symbol HF_Sym:L
- added U28: Z_{2}=2, symbol HF_Sym:UE
- added U29: C_{2} = 1, symbol HF_Sym:C
- added U30: L_{1} = 1, symbol HF_Sym:L
- added U31: L_{3} = 1, symbol HF_Sym:L
- added U32: Z_{1}=3/2, symbol HF_Sym:UE
- added U33: Z_{2}=3/10, symbol HF_Sym:UE
- added U34: Z_{3}=1/5, symbol HF_Sym:UE
- U3: value L=1 -> L_{2}=1/2
- U4: value L=1 -> L_{3}=1
- U5: value C=1 -> C_{1}=1
Connections:
- net at U1.: now also U2.
- net at U2.: now also R1.; no longer U1.
- net at U14.: now also U19.; no longer U18.
- net at U15.: now also U19.; no longer U14.
- net at U16.: now also U21.; no longer U14.
- net at R2., U6.: now also R3., U8.; no longer U7.
- net at R3., U8.: now also U7.; no longer R2., U6.
- net at U20.: now also U17.; no longer R7.
- net at U18.: now also U21.; no longer U17.
- new net: U1., U2.
- new net: U33., U34. (x2)
- new net: U14., U18.
- new net: U14., U15.
- new net: U14., U16.
- new net: U32., U33. (x2)
- new net: U10., U11., U13.
- new net: U10., U12., U9.
- new net: R2., U6., U7.
- new net: U29., U30., U31.
- new net: U29., U31.
- new net: U27., U28.
- new net: R7., U20.
- new net: R5., U13.
- new net: R1., U2.
- new net: U17., U18.
- new net: U18., U20.
- new net: U24., U26.
- new net: U22., U24.
- new net: R10., U28. (x2)
- new net: R6., U19.
- new net: R4., U12.
- now unconnected: U3., U4., U5.
Other:
- note added: "Z_{1}"
- note added: "Z_{2}"
- note added: "Z_{3}"

Commit message: Added Mischer
Parts:
- removed U10: L, symbol HF_Sym:L
- removed U13, U20: Z_{0}, symbol HF_Sym:UE
- removed U15, U17: L_{1}, symbol HF_Sym:L
- removed U16, U21: L/2, symbol HF_Sym:L
- added R11, R12, R13, R14: Z_{0}=1, symbol HF_Sym:R
- added R15: Y_{s}, symbol HF_Sym:R
- added R16: Y_{i}, symbol HF_Sym:R
- added U10: Z, symbol HF_Sym:UE
- added U13: C', symbol HF_Sym:C
- added U15: C_{2}=1/12, symbol HF_Sym:C
- added U16, U20: C_{21}, symbol HF_Sym:C
- added U17: ~, symbol HF_Sym:Trafo
- added U21: Z_{3}=2, symbol HF_Sym:UE
- added U35, U44: Z_{1}', symbol HF_Sym:UE
- added U36, U37, U39, U40, U43, U45, U48, U50: C_{21}', symbol HF_Sym:C
- added U38, U49: Z_{3}', symbol HF_Sym:UE
- added U41: n:1, symbol HF_Sym:Trafo
- added U42: 1:n, symbol HF_Sym:Trafo
- added U46: ~, symbol HF_Sym:CurrSource
- added U47: ~, symbol HF_Sym:Block
- added U51: C_{3}, symbol HF_Sym:C
- added U52: ~, symbol HF_Sym:ImpAdapt
- added U53: L_{3} = 1, symbol HF_Sym:L
- R4, R5, R6, R7: value Z_{0} -> Z_{0}=1
- U11: value C -> C'
- U12: value Z_{0} -> Z
- U14: value Z_{1} -> Z_{3}=2
- U18: value Z_{1} -> Z_{1}=2
- U19: value Z_{0} -> Z_{1}=2
Connections:
- net at U1.: now also U2.
- net at U2.: now also R1.; no longer U1.
- net at U34.: now also U33.
- net at U33.: now also U32.; no longer U34.
- net at U14.: now also U15.; no longer U18.
- net at U19.: now also U15.; no longer U14.
- net at U11.: now also U10.
- net at R2., U6.: now also R3., U8.; no longer U7.
- net at R3., U8.: now also U7.; no longer R2., U6.
- net at U29., U31.: no longer U30.
- net at U27.: now also U28.
- net at U28.: no longer U27.
- net at R7.: now also U14.
- net at R5.: now also U21.
- net at U18.: now also U21.
- net at U24.: now also U22.
- net at U26.: no longer U24.
- net at U22.: no longer U24.
- net at R4.: now also U18.; no longer U12.
- net at U12.: no longer R4.
- new net: U1., U2.
- new net: U33., U34.
- new net: R7., U14.
- new net: U14., U19.
- new net: U32., U33.
- new net: R2., U6., U7.
- new net: U29., U30., U31.
- new net: R12., U38.
- new net: R12., U40.
- new net: U43., U44.
- new net: R13., U43.
- new net: U10., U13.
- new net: U44., U45.
- new net: U45., U48.
- new net: U44., U49.
- new net: R13., U44.
- new net: R1., U2.
- new net: U24., U26.
- new net: R10., U28.
- new net: U48., U49.
- new net: U12., U9.
- new net: R4., U18.
- new net: U38., U40.
- new net: U38., U42.
- new net: U37., U38.
- new net: R11., U39.
- new net: R11., U35.
- new net: U16., U20.
- new net: U16., U21.
- new net: U41., U42. (x2)
- new net: U35., U41.
- new net: U36., U41.
- new net: U18., U20.
- new net: R16., U47. (x2)
- new net: R15., U46., U47. (x2)
- new net: R5., U21.
- new net: U37., U42.
- new net: R14., U49.
- new net: U49., U50.
- new net: U35., U39.
- new net: R6., U19.
- new net: U10., U17.
- new net: U11., U17.
- new net: R14., U50.
- new net: U35., U36.
- now unconnected: U12., U28.
Other:
- note added: "="
- note added: "> f_{s}"
- note added: "I_{i} <"
- note added: "I_{sg} >"
- note added: "I_{s} >"
- note added: "U_{i}↓"
- note added: "U_{s}↓"
- note added: "[G_{0} G_{1}] [G_{1}^{*}G_{0}]"
- note added: "f_{ZF}=f_{i} >"
- note added: "↓f_{LO}"
- note removed: "1"
